Commit message: commit before making new branch

File: EE3100704/examples/rsc/canine/urdf/canineV4_2.urdf (robot description, URDF)
Before this commit: robot canineV4, 14 links, 13 joints
Links:
- link HR_calf: mass 0.3639 -> 0.4049
- link HR_thigh: geometry collision cylinder length=0.024 radius=0.015; visual mesh filename=../meshes/HR_thigh_1.stl scale=0.001 0.001 0.001
